Commit message: Fix stale arm command type and record DDS discovery race
Two traps found while executing Task 3.

gazebo.xacro told the reader to command arm joints with std_msgs/msg/Double.
That type does not exist - the gz side is gz.msgs.Double and the bridge maps it
to std_msgs/Float64 - so following the comment silently does nothing. It is the
exact typo Task 3's type-validation step exists to catch, sitting in the file
that motivates the command.

`ros2 topic echo --once` intermittently reports a working publisher as absent:
each CLI call is a fresh node and sometimes gives up before discovering a
low-rate publisher. It reported a working bridge as broken. The plan now
requires a single long-lived rclpy subscriber for any "verify the topic
publishes" step.

Co-Authored-By: Claude Opus 5 <noreply@anthropic.com>

File: src/drivebase_description/urdf/gazebo.xacro (robot description, xacro)
@@ -111,5 +111,10 @@
     <!-- Targets come from the stow_* properties in drivebase.urdf.xacro. Command
          any joint at runtime with
-         `ros2 topic pub /arm/<joint>/position std_msgs/msg/Double ...`. -->
+         `ros2 topic pub /arm/<joint>/position std_msgs/msg/Float64 ...`.
+         Float64, NOT Double. These are gz transport topics carrying
+         gz.msgs.Double, and drivebase_sim's bridge.yaml maps them to
+         std_msgs/Float64 - there is no std_msgs/msg/Double, so the obvious
+         guess names a type that does not exist and the command silently does
+         nothing. -->
     <xacro:arm_joint_hold joint="shoulder_pan"  target="${stow_shoulder_pan}"/>
     <xacro:arm_joint_hold joint="shoulder_lift" target="${stow_shoulder_lift}"/>
