Commit message: Add Gazebo Harmonic simulation and power budget
drivebase_description:
- gazebo.xacro: DiffDrive (4-wheel skid steer), JointStatePublisher,
  IMU, NavSat (2.5m stddev per NEO-6M), 5x gpu_lidar as HC-SR04 cones
- gated behind use_sim xacro arg; hardware expansion unchanged
- DiffDrive tf parked on an unbridged topic so robot_localization can
  own odom->base_footprint

drivebase_sim (new):
- test_field.sdf: world-level sensor systems, spherical_coordinates
  for NavSat, barriers and posts as obstacles
- bridge.yaml: TwistStamped cmd_vel (verified against Jazzy Nav2 1.3.12)
- laserscan_to_range: collapses simulated cones to sensor_msgs/Range,
  matching what the real HC-SR04 driver will publish
- sim.launch.py, README with gotchas

docs/power_budget.md: load breakdown, two-pack architecture, motor
spec with sizing math, encoder rate justification for the Pico.

Verified in ros:jazzy container (software rendering):
- build + xacro + check_urdf pass for use_sim true and false
- rates: odom 50Hz, imu 100Hz, gps 5Hz, ultrasonic 2.9Hz
- front_center range 2.732m vs 2.75m predicted from world geometry
- odometry vs independent range ground truth: 0.000m error over 1.172m
- no odom->base_footprint publisher, 11 static transforms, 0 log errors

Co-Authored-By: Claude Opus 5 <noreply@anthropic.com>

File: src/drivebase_description/urdf/drivebase.urdf.xacro (robot description, xacro)
@@ -2,4 +2,8 @@
 <robot name="drivebase" xmlns:xacro="http://www.ros.org/wiki/xacro">
   <xacro:include filename="$(find drivebase_description)/urdf/inertia.xacro"/>
+  <!-- Adds Gazebo system plugins and simulated sensors. Off by default so the
+       same URDF drives real hardware unchanged. -->
+  <xacro:arg name="use_sim" default="false"/>
+  <xacro:property name="use_sim" value="$(arg use_sim)"/>
   <!-- ==================================================================
        GEOMETRY
@@ -182,3 +186,7 @@
   <xacro:ultrasonic name="front_midright" y="-0.060" yaw_deg="-25"/>
   <xacro:ultrasonic name="front_right"   y="-0.120" yaw_deg="-50"/>
+  <!-- Included last: gazebo.xacro reads the geometry properties above. -->
+  <xacro:if value="${use_sim}">
+    <xacro:include filename="$(find drivebase_description)/urdf/gazebo.xacro"/>
+  </xacro:if>
 </robot>

Commit message: Square the wheel layout, mount the SO-101, fix mesh and sensor geometry
Geometry (per measured chassis):
- wheelbase 150 -> 430, chassis 350 -> 430 square. Front axle now at
  x=+215, ahead of the arm mount at +155, so the arm loads the wheelbase
  instead of cantilevering past it.
- ultrasonic band raised 50 -> 140mm (200mm above ground). The square
  wheelbase puts front wheels 60mm ahead of the chassis face; at hub
  height the outer cones read a permanent 0.08-0.09m obstacle (measured).
  Raising clears the 120mm wheel tops and keeps the full +-50deg fan.

so101_description (new):
- upstream URDF vendored + 13 meshes (~15MB) for reproducibility
- vendor_so101.py generates a prefixed xacro macro; collision geometry
  replaced with per-mesh bounding boxes so Gazebo isn't computing
  mesh-mesh contacts on 0.5-2.6MB STLs every step
- prefixing is required: upstream's root link is also called base_link

Arm integration:
- attached at arm_mount_link behind use_arm (default true)
- gz JointPositionController per joint holds the stow pose; without it
  the arm collapses on the first step and shifts the base CoM
- stow pose found by sweeping poses in-sim and reading tf, not by
  hand kinematics: gripper x=+0.114 z=+0.600, inside the footprint,
  vs x=+0.554 at the all-zero pose
- GZ_SIM_RESOURCE_PATH set in sim.launch.py; without it gz rewrites
  package:// to model://, fails to find meshes, and the arm renders
  invisible while remaining present in physics

Also: ultrasonic ray visualisation on by default.

Verified in ros:jazzy (software rendering), 0 log errors:
- all 3 xacro variants pass check_urdf
- ultrasonics clear (4.0m), front_center 2.689m vs 2.710m predicted
- drive 1.152m over 4s at 0.3m/s, stops clean

Known blocking issue recorded in docs/power_budget.md: gripper bottoms
out 389mm above ground on the top-plane mount and cannot reach litter.

Co-Authored-By: Claude Opus 5 <noreply@anthropic.com>

File: src/drivebase_description/urdf/drivebase.urdf.xacro (robot description, xacro)
@@ -6,4 +6,33 @@
   <xacro:arg name="use_sim" default="false"/>
   <xacro:property name="use_sim" value="$(arg use_sim)"/>
+  <!-- Mounts the SO-101 on the top plane. Off gives a bare drivebase, which is
+       useful for isolating whether a handling problem is the arm's mass or the
+       base itself. -->
+  <xacro:arg name="use_arm" default="true"/>
+  <xacro:property name="use_arm" value="$(arg use_arm)"/>
+  <xacro:if value="${use_arm}">
+    <xacro:include filename="$(find so101_description)/urdf/so101_macro.xacro"/>
+  </xacro:if>
+  <!-- Draw the ultrasonic cones in the Gazebo GUI. On by default: seeing which
+       cone caught an obstacle is most of the value of running the sim at all. -->
+  <xacro:arg name="show_sensor_rays" default="true"/>
+  <xacro:property name="show_sensor_rays" value="$(arg show_sensor_rays)"/>
+  <!-- Arm stow pose, radians. PROVISIONAL - the arm team owns the real one.
+       It matters to navigation, not just aesthetics: at the all-zero pose the
+       gripper reaches ~290 mm past the chassis face, roughly 200 mm outside the
+       robot's footprint circle, so Nav2 would plan paths that clip the arm
+       through obstacles. Stowing it inside the footprint is what lets the
+       footprint stay the chassis. -->
+       Found by sweeping poses in the running simulator and reading
+       base_link -> arm_gripper_frame_link from tf, not by hand-solved kinematics.
+       Measured result: gripper at x=+0.110, z=+0.592 - 105 mm inside the chassis
+       face and standing clear above the roof, versus x=+0.554 at the all-zero
+       pose. Joint use stays off the hard limits (lift 83%, elbow 92%, wrist 66%). -->
+  <xacro:property name="stow_shoulder_pan"  value="0.0"/>
+  <xacro:property name="stow_shoulder_lift" value="1.45"/>
+  <xacro:property name="stow_elbow_flex"    value="1.55"/>
+  <xacro:property name="stow_wrist_flex"    value="1.10"/>
+  <xacro:property name="stow_wrist_roll"    value="0.0"/>
+  <xacro:property name="stow_gripper"       value="0.0"/>
   <!-- ==================================================================
        GEOMETRY
@@ -15,9 +44,14 @@
   <xacro:property name="wheel_width"     value="0.040"/>   <!-- ESTIMATE -->
   <xacro:property name="track"           value="0.430"/>   <!-- left<->right -->
-  <xacro:property name="wheelbase"       value="0.150"/>   <!-- front<->rear -->
-  <!-- Chassis body. ESTIMATES until the print is measured. -->
-  <xacro:property name="chassis_length"  value="0.350"/>
-  <xacro:property name="chassis_width"   value="0.350"/>
-  <xacro:property name="chassis_height"  value="0.350"/>
+  <!-- Square wheel layout. Puts the front axle at x=+215, well ahead of the arm
+       mount at x=+115, so the arm loads the wheelbase instead of cantilevering
+       past it. Side effect: the wheels now protrude ~100 mm beyond the chassis
+       front face - see the ultrasonic placement note below. -->
+  <xacro:property name="wheelbase"       value="0.430"/>   <!-- front<->rear -->
+  <!-- Chassis body. Footprint is measured; height is still an ESTIMATE carried
+       over from "cube chassis". -->
+  <xacro:property name="chassis_length"  value="0.430"/>
+  <xacro:property name="chassis_width"   value="0.430"/>
+  <xacro:property name="chassis_height"  value="0.430"/>
   <xacro:property name="ground_clearance" value="0.030"/>
   <!-- Masses. ESTIMATES. Only matter for simulation dynamics. -->
@@ -165,5 +199,12 @@
        the drive corridor. Mounted low so the arm and its payload stay out
        of the cones. -->
-  <xacro:property name="us_z" value="0.050"/>
+  <!-- 0.14 above base_link = 200 mm above ground, clearing the 120 mm wheel tops
+       by 80 mm. At 0.05 the outer cones looked straight into the front wheels and
+       reported a permanent 0.08-0.09 m obstacle (measured, before this change) -
+       the square wheelbase puts the front wheels 60 mm ahead of the chassis face,
+       so anything at hub height sees them. Raising the band clears the wheels
+       geometrically and keeps the full +-50 deg fan; narrowing the fan instead
+       would have cost real coverage. -->
+  <xacro:property name="us_z" value="0.140"/>
   <xacro:macro name="ultrasonic" params="name y yaw_deg">
     <link name="ultrasonic_${name}_link">
@@ -186,4 +227,14 @@
   <xacro:ultrasonic name="front_midright" y="-0.060" yaw_deg="-25"/>
   <xacro:ultrasonic name="front_right"   y="-0.120" yaw_deg="-50"/>
+  <!-- ==================================================================
+       ARM
+       SO-101 on the top plane, its own base frame already Z-up so the mount
+       transform is identity.
+       ================================================================== -->
+  <xacro:if value="${use_arm}">
+    <xacro:so101 prefix="arm_" parent="arm_mount_link">
+      <origin xyz="0 0 0" rpy="0 0 0"/>
+    </xacro:so101>
+  </xacro:if>
   <!-- Included last: gazebo.xacro reads the geometry properties above. -->
   <xacro:if value="${use_sim}">

File: src/drivebase_description/urdf/gazebo.xacro (robot description, xacro)
@@ -52,16 +52,49 @@
             name="gz::sim::systems::JointStatePublisher">
       <topic>${gz_prefix}/joint_state</topic>
-      <!-- KNOWN WART: this publishes every physics step (~1 kHz) and gz's
+      <!-- No <joint_name> entries: publishes every joint, so the arm's six come
+           along automatically and robot_state_publisher can build arm tf.
+           KNOWN WART: this publishes every physics step (~1 kHz) and gz's
            JointStatePublisher has no rate limit - <update_rate> here is silently
            ignored (measured: still 980 Hz with it set). Tolerated because it is
-           sim-only and only drives wheel-spin visuals; nothing downstream reads
-           wheel angle. On hardware the Pico publishes joint states at a sane
-           rate instead. Revisit only if it hurts real-time factor. -->
-      <joint_name>front_left_wheel_joint</joint_name>
-      <joint_name>front_right_wheel_joint</joint_name>
-      <joint_name>rear_left_wheel_joint</joint_name>
-      <joint_name>rear_right_wheel_joint</joint_name>
+           sim-only. On hardware the Pico publishes wheel state and the Feetech
+           bus publishes arm state, both at sane rates. -->
     </plugin>
   </gazebo>
+  <!-- ==================================================================
+       ARM JOINT HOLD
+       Without a controller the arm joints are free and the arm collapses under
+       gravity on the first step, which also shifts the base's centre of mass and
+       corrupts any handling measurement. Real STS3215 servos hold position, so
+       modelling them as position-controlled is both more correct and more stable.
+       This is what the ~11 W idle arm draw in docs/power_budget.md pays for.
+       ================================================================== -->
+  <xacro:if value="${use_arm}">
+    <xacro:macro name="arm_joint_hold" params="joint target:=0">
+      <gazebo>
+        <plugin filename="gz-sim-joint-position-controller-system"
+                name="gz::sim::systems::JointPositionController">
+          <joint_name>arm_${joint}</joint_name>
+          <topic>/arm/${joint}/position</topic>
+          <initial_position>${target}</initial_position>
+          <p_gain>4.0</p_gain>
+          <i_gain>0.05</i_gain>
+          <d_gain>0.15</d_gain>
+          <i_max>1.0</i_max>
+          <i_min>-1.0</i_min>
+          <cmd_max>10.0</cmd_max>
+          <cmd_min>-10.0</cmd_min>
+        </plugin>
+      </gazebo>
+    </xacro:macro>
+    <!-- Targets come from the stow_* properties in drivebase.urdf.xacro. Command
+         any joint at runtime with
+         `ros2 topic pub /arm/<joint>/position std_msgs/msg/Double ...`. -->
+    <xacro:arm_joint_hold joint="shoulder_pan"  target="${stow_shoulder_pan}"/>
+    <xacro:arm_joint_hold joint="shoulder_lift" target="${stow_shoulder_lift}"/>
+    <xacro:arm_joint_hold joint="elbow_flex"    target="${stow_elbow_flex}"/>
+    <xacro:arm_joint_hold joint="wrist_flex"    target="${stow_wrist_flex}"/>
+    <xacro:arm_joint_hold joint="wrist_roll"    target="${stow_wrist_roll}"/>
+    <xacro:arm_joint_hold joint="gripper"       target="${stow_gripper}"/>
+  </xacro:if>
   <!-- ==================================================================
        WHEEL CONTACT
@@ -147,5 +180,7 @@
         <always_on>1</always_on>
         <update_rate>3</update_rate>
-        <visualize>false</visualize>
+        <!-- Draws the cones as visible rays in the Gazebo GUI, so you can watch
+             them hit and clear obstacles. Costs nothing headless. -->
+        <visualize>${show_sensor_rays}</visualize>
         <topic>/ultrasonic/${name}/scan</topic>
         <gz_frame_id>ultrasonic_${name}_link</gz_frame_id>

Commit message: Relocate arm to front face, add local EKF, wire RViz into sim launch
Arm mount (corrects an earlier wrong measurement):
- I previously reported the gripper bottoming out at 389mm above ground.
  That was wrong - the sweep folded the elbow in every downward attempt, so
  the arm was never actually extended. With elbow/wrist at zero the real
  minimum from the top plane was 241mm.
- Useful figure is reach below mount: 219mm. Moved the mount from the top
  plane (460mm) to the front face at 260mm, giving a gripper minimum of
  41mm above ground - within grasping range of litter.
- Mounted on the face rather than bracketed ahead of it, so the base plate
  protrudes ~55mm, less than the wheels' 60mm, keeping the Nav2 footprint
  as the wheel envelope.
- Stow pose re-measured for the new mount: folded, gripper 230mm up.
  Folding backward from a front mount drives the gripper into the body, so
  up-and-forward is the available direction.

drivebase_localization (new):
- local EKF, odom -> base_footprint, 30Hz
- fuses wheel vx + IMU yaw/yaw-rate; deliberately NOT wheel yaw

  Measured against Gazebo ground truth, commanding 0.4rad/s for 3s:
    ground truth      44.97 deg
    EKF (IMU)         45.0  deg   correct
    wheel-model odom  69.0  deg   over-reports 1.53x

  So fusing wheel yaw would have put heading 53% wrong after one turn, and
  only ~65% of commanded rotation is achieved - the rest lost to scrub.
  Factor is state-dependent (1.94x seen after translating), so it is a
  hardware calibration item, not a constant.

sim launch:
- ekf:=true (default) and rviz:=true args; one command brings up everything
- RViz shows EKF pose against raw wheel odom so the scrub gap is visible

Verified in ros:jazzy, 0 errors: all topics live from a single launch,
exactly one publisher of odom->base_footprint. After a 4s drive+turn,
EKF x within 7mm of ground truth, y off by 99mm - dead-reckoning drift
that the global GPS-corrected filter is meant to correct.

Co-Authored-By: Claude Opus 5 <noreply@anthropic.com>

File: src/drivebase_description/urdf/drivebase.urdf.xacro (robot description, xacro)
@@ -24,11 +24,14 @@
        through obstacles. Stowing it inside the footprint is what lets the
        footprint stay the chassis. -->
-       Found by sweeping poses in the running simulator and reading
-       base_link -> arm_gripper_frame_link from tf, not by hand-solved kinematics.
-       Measured result: gripper at x=+0.110, z=+0.592 - 105 mm inside the chassis
-       face and standing clear above the roof, versus x=+0.554 at the all-zero
-       pose. Joint use stays off the hard limits (lift 83%, elbow 92%, wrist 66%). -->
+       Measured in the running simulator via base_link -> arm_gripper_frame_link,
+       not hand-solved: gripper at x=+0.309, z=+0.170 (230 mm above ground). Folded
+       rather than extended, gripper carried clear of the ground, and every joint
+       off its hard limit (lift 69%, elbow 92%, wrist 66%).
+       Only ~34 mm past the wheel line, so the Nav2 footprint stays the wheel
+       envelope. Not tucked fully inside the chassis - folding backward from a
+       front-face mount drives the gripper into the body, so up-and-forward is the
+       available direction. -->
   <xacro:property name="stow_shoulder_pan"  value="0.0"/>
-  <xacro:property name="stow_shoulder_lift" value="1.45"/>
+  <xacro:property name="stow_shoulder_lift" value="-1.20"/>
   <xacro:property name="stow_elbow_flex"    value="1.55"/>
   <xacro:property name="stow_wrist_flex"    value="1.10"/>
@@ -185,7 +188,14 @@
     <origin xyz="0 0 0" rpy="${-pi/2} 0 ${-pi/2}"/>
   </joint>
-  <!-- Arm mount. SO101 sits vertically on the top plane near the front
-       edge. This frame is where the SO101's own URDF gets attached; it is
-       not the arm itself. -->
+  <!-- Arm mount. Bolted to the front face with the base plate horizontal, so the
+       arm stands up from it and reaches forward and down.
+       HEIGHT IS LOAD-BEARING, not cosmetic. Measured in simulation: the SO-101
+       reaches 219 mm below its own mount (gripper 241 mm above ground when
+       mounted at 460 mm, elbow and wrist extended). Litter on the ground needs
+       the gripper near 30-40 mm, so the mount has to sit around 250-260 mm.
+       260 mm also clears the ultrasonic band at 200 mm by 17 mm once the base
+       link's own 87 mm height is accounted for.
+       On the top plane (460 mm) the arm could not reach the ground at all. -->
+  <xacro:property name="arm_mount_z" value="0.200"/>  <!-- 260 mm above ground -->
   <link name="arm_mount_link">
     <xacro:sensor_inertia/>
@@ -194,5 +204,8 @@
     <parent link="base_link"/>
     <child  link="arm_mount_link"/>
-    <origin xyz="${front_face_x - 0.060} 0 ${top_plane_z}" rpy="0 0 0"/>
+    <!-- On the face, not bracketed ahead of it: the base plate then protrudes
+         ~55 mm, less than the wheels' 60 mm, so the Nav2 footprint stays the
+         wheel envelope instead of growing to include the arm. -->
+    <origin xyz="${front_face_x} 0 ${arm_mount_z}" rpy="0 0 0"/>
   </joint>
   <!-- Ultrasonic band. Five sensors across the front face, fanned to cover
