Commit message: Add scripted_drive measurement rig; measure turn drift and track factor
The ad-hoc shell harness used for earlier measurements was unreliable in five
ways, most seriously that backgrounded `ros2 topic pub` survived kill and
competed, so a "square" test recorded clean while the robot drove straight.
drivebase_sim/scripted_drive.py replaces it: one process owning one publisher,
one timer sampling all sources at the same instant, sim-time deadlines, and legs
that terminate on measured progress rather than elapsed time. Turns close the
loop on ground truth so every run drives the same real path.

Ground truth now comes from gz OdometryPublisher (the model's true world pose),
bridged to /gz/ground_truth - deliberately never onto /tf, which would displace
the estimate being measured. First tried bridging dynamic_pose/info, but the
Pose_V -> TFMessage conversion leaves child_frame_id EMPTY, so the robot cannot
be identified in the pose array.

MEASURED

  A 90 deg turn costs ~0.35 m of local-EKF position error.
  Twenty metres of straight driving costs essentially nothing.

Nine runs over three paths whose lengths differ nearly 7x (3.0, 5.5, 20.4 m) all
show 0.347-0.351 m of error, because all nine completed exactly one 90 deg
rotation. Distance is not the variable; rotation is. That resolves the earlier
contradiction between ~0.5% error on straight runs and ~9% per metre on a Nav2
run with two turns.

  Effective-track factor: 1.742x, stdev 0.025, n=6.

Stable across lateral friction from 0.15 to 0.6, confirming it is kinematic
rather than frictional. Supersedes the 1.53x and 1.94x single samples taken with
the old harness. Folded into gazebo.xacro and ekf_local.yaml as documentation;
wheel_separation stays at the physical track deliberately, so the sim keeps the
same bias the real robot has.

NOT MEASURED, AND WHY

Linearity of turn cost. The simulated robot cannot rotate in place more than once
per run: the first rotation succeeds, every later one leaves the body stationary
while the wheel joints spin (measured: odom_yaw +279 deg, true_yaw 0.0 deg).
Ruled out by experiment - commanded angular velocity (0.5/0.8/1.2), the arm
(arm:=false fails too), lateral friction (0.6/0.3/0.15), and translation between
turns (twoturns path). Remaining hypothesis is that DiffDrive commands joint
velocity with no torque limit, so contacts simply slip and friction force is
independent of commanded speed - which is why raising angular velocity changed
nothing.

So no sim-derived claim about repeated turning is trustworthy, including the
earlier "~65% of commanded rotation achieved". Nav2's obstacle-avoidance results
stand: RPP arcs rather than point-turns.

Also fixed a malformed comment block in drivebase.urdf.xacro that I introduced
with the stow-pose edit - it closed early, leaving nine lines of prose as
character data with a stray "-->". It parsed only because XML tolerates text
inside an element, so URDF silently ignored it and every build passed.

New: wheel_mu1/wheel_mu2 and arm:= launch args for sweeping the contact model,
scripts/analyse_drift.py, docs/localization_accuracy.md.

Co-Authored-By: Claude Opus 5 <noreply@anthropic.com>

File: src/drivebase_description/urdf/drivebase.urdf.xacro (robot description, xacro)
@@ -14,4 +14,10 @@
     <xacro:include filename="$(find so101_description)/urdf/so101_macro.xacro"/>
   </xacro:if>
+  <!-- Wheel contact friction, exposed so the contact model can be swept. The
+       simulated robot cannot rotate in place reliably - only the first rotation
+       of a run succeeds - and lateral friction is the prime suspect. See
+       docs/localization_accuracy.md. -->
+  <xacro:arg name="wheel_mu1" default="1.0"/>
+  <xacro:arg name="wheel_mu2" default="0.6"/>
   <!-- Draw the ultrasonic cones in the Gazebo GUI. On by default: seeing which
        cone caught an obstacle is most of the value of running the sim at all. -->
@@ -23,5 +29,5 @@
        robot's footprint circle, so Nav2 would plan paths that clip the arm
        through obstacles. Stowing it inside the footprint is what lets the
-       footprint stay the chassis. -->
+       footprint stay the chassis.
        Measured in the running simulator via base_link -> arm_gripper_frame_link,
        not hand-solved: gripper at x=+0.309, z=+0.170 (230 mm above ground). Folded

File: src/drivebase_description/urdf/gazebo.xacro (robot description, xacro)
@@ -32,7 +32,11 @@
            the same bias in the same direction, which is exactly why the EKF must
            take yaw from the IMU rather than the wheels. Compensating it means
-           using an effective track wider than the physical one (typically
-           1.5-1.8x). Left at the true value deliberately - that factor gets
-           measured on hardware, not guessed here. -->
+           using an effective track wider than the physical one. MEASURED in
+           simulation over 6 clean turns: 1.742x (stdev 0.025), i.e. an effective
+           wheel_separation of 0.749 m. See docs/localization_accuracy.md.
+           Left at the physical track deliberately: the simulation should carry
+           the same bias the real robot has, which is what forces the EKF to take
+           yaw from the IMU rather than the wheels. Correcting it here would hide
+           the very effect the EKF exists to handle. -->
       <wheel_separation>${track}</wheel_separation>
       <wheel_radius>${wheel_radius}</wheel_radius>
@@ -48,4 +52,22 @@
       <tf_topic>${gz_prefix}/unused_tf</tf_topic>
       <max_linear_acceleration>1.5</max_linear_acceleration>
+    </plugin>
+    <!-- GROUND TRUTH, for measuring the estimators against. Reads the model's
+         true world pose (WorldPoseTag), so it is not a simulated sensor and
+         carries no error - gaussian_noise is deliberately left unset.
+         Chosen over bridging /world/.../dynamic_pose/info: that arrives as a
+         Pose_V, and the bridge's TFMessage conversion leaves child_frame_id
+         EMPTY (measured), so there is no way to tell which entity is the robot.
+         tf_topic is parked unbridged for the same reason as DiffDrive's - ground
+         truth must never reach /tf, or it would displace the estimate being
+         measured. -->
+    <plugin filename="gz-sim-odometry-publisher-system"
+            name="gz::sim::systems::OdometryPublisher">
+      <odom_topic>${gz_prefix}/ground_truth</odom_topic>
+      <odom_frame>truth_origin</odom_frame>
+      <robot_base_frame>base_footprint</robot_base_frame>
+      <odom_publish_frequency>50</odom_publish_frequency>
+      <dimensions>2</dimensions>
+      <tf_topic>${gz_prefix}/unused_truth_tf</tf_topic>
     </plugin>
     <plugin filename="gz-sim-joint-state-publisher-system"
@@ -105,8 +127,10 @@
        measured hardware.
        ================================================================== -->
+  <xacro:property name="wheel_mu1" value="$(arg wheel_mu1)"/>
+  <xacro:property name="wheel_mu2" value="$(arg wheel_mu2)"/>
   <xacro:macro name="wheel_surface" params="link">
     <gazebo reference="${link}">
-      <mu1>1.0</mu1>
-      <mu2>0.6</mu2>
+      <mu1>${wheel_mu1}</mu1>
+      <mu2>${wheel_mu2}</mu2>
     </gazebo>
   </xacro:macro>

Commit message: Add eye-in-hand sensor pod frames on arm_wrist_link
Co-Authored-By: Claude Opus 5 <noreply@anthropic.com>

File: src/drivebase_description/urdf/drivebase.urdf.xacro (robot description, xacro)
@@ -255,4 +255,42 @@
       <origin xyz="0 0 0" rpy="0 0 0"/>
     </xacro:so101>
+    <!-- Sensor pod: camera + ToF, eye-in-hand.
+         Mounted on arm_wrist_link, which is BEFORE wrist_roll in the chain. The
+         camera therefore never rolls, so the image up-vector is fixed and the
+         harness crosses four moving joints rather than five. See
+         docs/superpowers/specs/2026-07-30-behaviour-coordinator-design.md §4.
+         CO-LOCATION IS LOAD-BEARING. A 20 mm camera-to-ToF separation at 80 mm
+         range is a large angular disagreement - the ToF can be reading past the
+         target while the camera reports it centred. These offsets are a
+         placeholder until the physical pod exists; they must be remeasured, and
+         must never be assumed zero. -->
+    <xacro:property name="pod_camera_xyz" value="0.010 0.0 0.030"/>
+    <xacro:property name="pod_camera_rpy" value="0 0 0"/>
+    <xacro:property name="pod_tof_xyz"    value="0.010 0.0 0.015"/>
+    <link name="pod_camera_link">
+      <xacro:sensor_inertia/>
+    </link>
+    <joint name="pod_camera_joint" type="fixed">
+      <parent link="arm_wrist_link"/>
+      <child  link="pod_camera_link"/>
+      <origin xyz="${pod_camera_xyz}" rpy="${pod_camera_rpy}"/>
+    </joint>
+    <!-- ROS optical convention: z forward, x right, y down. Image pipelines and
+         the ray projection in drivebase_behaviour/localisation.py both assume
+         it. Same rotation the chassis camera_optical_joint uses. -->
+    <link name="pod_camera_optical_frame"/>
+    <joint name="pod_camera_optical_joint" type="fixed">
+      <parent link="pod_camera_link"/>
+      <child  link="pod_camera_optical_frame"/>
+      <origin xyz="0 0 0" rpy="${-pi/2} 0 ${-pi/2}"/>
+    </joint>
+    <link name="pod_tof_link">
+      <xacro:sensor_inertia/>
+    </link>
+    <joint name="pod_tof_joint" type="fixed">
+      <parent link="arm_wrist_link"/>
+      <child  link="pod_tof_link"/>
+      <origin xyz="${pod_tof_xyz}" rpy="0 0 0"/>
+    </joint>
   </xacro:if>
   <!-- Included last: gazebo.xacro reads the geometry properties above. -->

Commit message: Keep the sensor pod at rpy 0 0 0, and find the confirm pose
Task 5b's premise was that the pod's 87.2 deg offset from the gripper's
approach axis is what stops CONFIRMING from working, and that rotating the
mount to close it would let some arm pose view the 0.287-0.481 m grasp window.
Both halves are wrong, and the second one is wrong in a useful direction.

Aiming the pod at the gripper blinds it. Two mounts were built and driven:
the prescribed rpy 0 -0.1145 -1.5213 (angle check passes at 0.024 deg) read a
constant 0.058 m across 31 poses, and rpy 0 0.0402 -1.6374 from a mount moved
0.030/0.040 outboard read 0.089 m across 44. Both persist at poses whose ray
points at open sky, where an unobstructed beam must return the sensor's
4.000 m max, and across wrist_roll -2.5..+2.5 rad and both gripper openings.
The pod sits at the root of a 160 mm gripper, so any aim at the grasp point
looks lengthwise down the gripper body; ray-casting the visual meshes shows
clearing the castings by 60 mm costs 80 mm of displacement from the grasp axis.
No rotation fixes that. Reverted to rpy 0 0 0, where the beam clears the
nearest casting by 69.5 deg and the sky check returns exactly 4.000 m.

But the grasp window IS viewable, and always was. Task 5 concluded no pose
could see it after 210 poses; it never drove the corner where it happens -
strongly negative wrist_flex against positive shoulder_lift, which none of its
sweeps paired. Confirm pose: pan 0, lift 0.9, elbow 0.46, wrist_flex -1.40.
The beam lands at x = 0.392 m, mid-window, measuring 0.2716 m against a
tf-only prediction of 0.2715 m. All 26 confirm candidates driven agreed with
prediction to better than 0.7%. The pose does not hold the gripper over the
target - it cannot, given the 87 deg offset - so CONFIRMING ranges and images
the target from there and the approach stays a separate open-loop motion.

Search pose unchanged at lift -1.4, elbow 0.0, wrist_flex 0.4: 1.138 m of
ground against a prediction of 1.118 m, gripper tucked to x = 0.267 m. Task 5
recorded 1.080/1.062 for the same command; the gap is droop, and both runs are
internally consistent, so the range is repeatable only to about 5%.

pod_camera_rpy becomes pod_aim_rpy and is now shared by both pod joints, which
previously had it hardcoded separately - they must stay boresighted.

The three measurement harnesses are committed this time. Task 5 threw its
sweep away and rebuilding it cost most of this task.

Also corrects PROGRESS.md's note that /tof/pod is RELIABLE: it is published
with qos_profile_sensor_data, so a RELIABLE subscriber silently receives
nothing.

Co-Authored-By: Claude Opus 5 <noreply@anthropic.com>

File: src/drivebase_description/urdf/drivebase.urdf.xacro (robot description, xacro)
@@ -266,6 +266,29 @@
          must never be assumed zero. -->
     <xacro:property name="pod_camera_xyz" value="0.010 0.0 0.030"/>
-    <xacro:property name="pod_camera_rpy" value="0 0 0"/>
     <xacro:property name="pod_tof_xyz"    value="0.010 0.0 0.015"/>
+    <!-- DO NOT ROTATE THIS TO POINT AT THE GRIPPER. It was tried, twice, and
+         both attempts blinded the sensor outright. Keeping zero is a measured
+         result, not the absence of one.
+         arm_wrist_link's +X genuinely does not point at the gripper: the SO-101
+         puts arm_gripper_frame_link at (0.00790, -0.15923, 0.01832) here,
+         essentially along -Y, 87.2 degrees off +X. Aiming the pod along that
+         approach axis looks like the obvious correction. It is not, because the
+         gripper body itself runs from this link out to the jaws, so that line of
+         sight is straight down it:
+           rpy 0 -0.1145 -1.5213, offsets as above ....... 0.058 m at 31 poses
+           rpy 0  0.0402 -1.6374, offsets 0.030/0.040 .... 0.089 m at 44 poses
+         Both figures are constant to +-3 mm across poses whose geometry differs
+         completely, and both persist at poses whose ray points at open sky,
+         where an unobstructed beam must return the sensor's 4.000 m max. That is
+         the robot's own castings, at every arm pose, every wrist_roll from -2.5
+         to +2.5 rad, and both gripper openings.
+         At rpy 0 0 0 the beam clears the castings by 69.5 degrees and the sky
+         check returns exactly 4.000 m. See docs/arm_workspace.md §3 for the
+         search and confirm poses this supports, and scripts/pod_aim_search.py
+         for the sweep over every mounting orientation.
+         Shared by both pod joints so they cannot drift apart: the camera's view
+         axis and the ToF ray agree to 4 decimal places at every pose measured,
+         and the localisation maths assumes exactly that. -->
+    <xacro:property name="pod_aim_rpy" value="0 0 0"/>
     <link name="pod_camera_link">
       <xacro:sensor_inertia/>
@@ -274,5 +297,5 @@
       <parent link="arm_wrist_link"/>
       <child  link="pod_camera_link"/>
-      <origin xyz="${pod_camera_xyz}" rpy="${pod_camera_rpy}"/>
+      <origin xyz="${pod_camera_xyz}" rpy="${pod_aim_rpy}"/>
     </joint>
     <!-- ROS optical convention: z forward, x right, y down. Image pipelines and
@@ -291,5 +314,5 @@
       <parent link="arm_wrist_link"/>
       <child  link="pod_tof_link"/>
-      <origin xyz="${pod_tof_xyz}" rpy="0 0 0"/>
+      <origin xyz="${pod_tof_xyz}" rpy="${pod_aim_rpy}"/>
     </joint>
   </xacro:if>

Commit message: Fix the rotation bug with gz-sim-wheel-slip-system, and re-measure everything
STATUS.md issue 1, closed. Candidate 1 was the right one.

dartsim takes a single friction coefficient and does not implement the
anisotropic mu1/mu2 split, so the lateral value in gazebo.xacro was discarded on
load with no warning. The robot ran effectively isotropic at mu1 1.0 against a
0.9 ground plane and slid instead of rotating. gz-sim-wheel-slip-system supplies
the anisotropy dartsim throws away, modelling slip rather than blunting friction
globally the way lowering mu1 does — so mu1 stays at 1.0.

  twoturns   aborted on turn 1     -> completes, 181 deg, 0.10 m scrub
  square5    aborted at corner 1   -> completes, 20.3 m, 453 deg

For comparison the mu1:=0.35 workaround got twoturns through at 0.42 m of
scrub. The slip model does it at 0.10 m without touching mu1.

THE PART THAT MATTERS MORE THAN THE FIX: two documented figures were wrong.

The effective-track factor moved from 1.742x (n=6) to 2.112x (n=10, stdev
0.008) — up, because the wheels now scrub freely instead of the body sliding.
That also retires the claim that it was "stable across lateral-friction values
from 0.15 to 0.6, so it is kinematic not frictional". It was stable because
those values were being discarded. It moved 21% as soon as the contact model
really changed.

And the headline turn-cost figure was measuring the bug itself. "~0.35 m of
error per 90 degrees" was largely the body sliding 0.156 m through a turn it
never completed. A full five-turn 20 m square now drifts 0.035 m — a factor of
~50. Updated in localization_accuracy.md, STATUS.md, ekf_local.yaml and the
README, with the old numbers kept visible so the change is auditable.

The design conclusion is unchanged but now rests on different evidence: aim the
arm with the camera because GPS bounds error at 1.4-5.6 m, because the simulated
IMU is better than any real part, and because no contact model here has been
checked against hardware — not because turns cost 0.35 m.

Also fixes scripts/analyse_drift.py, which was silently discarding every turn.
It diffed yaw endpoints, which cannot represent a rotation past pi, so it
carried a wheel_delta > 2.8 guard — and the new over-report pushed all ten turns
past it. It reported "no usable turns found" for a run where every turn was
clean. Now accumulates wrapped step-to-step differences, which has no ceiling.

slip_lateral 1.0 has no more hardware justification than mu1 0.35 did. It is a
value that makes the sim behave like a skid-steer rather than a sledge, and it
needs re-measuring against real tyres.

Co-Authored-By: Claude Opus 5 <noreply@anthropic.com>

File: src/drivebase_description/urdf/drivebase.urdf.xacro (robot description, xacro)
@@ -20,4 +20,14 @@
   <xacro:arg name="wheel_mu1" default="1.0"/>
   <xacro:arg name="wheel_mu2" default="0.6"/>
+  <!-- Wheel slip model. dartsim takes a single friction coefficient and
+       discards the mu1/mu2 split, so anisotropy has to come from somewhere
+       else; gz-sim-wheel-slip-system is where. Compliance is (m/s)/N and is
+       divided by wheel_normal_force internally, so these are per-unit-force
+       figures. Lateral non-zero lets the tyres scrub during a point turn;
+       longitudinal near zero keeps them gripping for drive. Exposed so the
+       contact model stays sweepable the way wheel_mu1 is. -->
+  <xacro:arg name="wheel_slip" default="true"/>
+  <xacro:arg name="slip_lateral" default="1.0"/>
+  <xacro:arg name="slip_longitudinal" default="0.0"/>
   <!-- Draw the ultrasonic cones in the Gazebo GUI. On by default: seeing which
        cone caught an obstacle is most of the value of running the sim at all. -->

File: src/drivebase_description/urdf/gazebo.xacro (robot description, xacro)
@@ -215,4 +215,40 @@
   <xacro:wheel_surface link="rear_right_wheel_link"/>
   <!-- ==================================================================
+       WHEEL SLIP
+       The mu1/mu2 pair above maps to ODE's friction element. gz-sim's default
+       physics engine is dartsim, which takes ONE friction coefficient and
+       silently discards the lateral value on load. That is why sweeping
+       wheel_mu2 across 0.6/0.3/0.15 changed nothing: the parameter had no
+       effect to have, and the robot ran effectively isotropic at mu1 against
+       a 0.9 ground plane — the "isotropic high friction makes a skid-steer
+       refuse to rotate" case the comment above warns about.
+       This plugin is where the anisotropy actually comes from. It models slip
+       properly rather than blunting friction globally, which is what lowering
+       mu1 does — and lowering mu1 changes how much the tyres scrub, which
+       invalidates every measured figure in docs/localization_accuracy.md.
+       wheel_normal_force is the static load per wheel: 10.342 kg total mass
+       (summed from the URDF) x 9.81 / 4 = 25.4 N.
+       ================================================================== -->
+  <xacro:property name="wheel_slip" value="$(arg wheel_slip)"/>
+  <xacro:if value="${wheel_slip}">
+    <gazebo>
+      <plugin filename="gz-sim-wheel-slip-system"
+              name="gz::sim::systems::WheelSlip">
+        <xacro:macro name="slip_wheel" params="link">
+          <wheel link_name="${link}">
+            <slip_compliance_lateral>$(arg slip_lateral)</slip_compliance_lateral>
+            <slip_compliance_longitudinal>$(arg slip_longitudinal)</slip_compliance_longitudinal>
+            <wheel_normal_force>25.4</wheel_normal_force>
+            <wheel_radius>${wheel_radius}</wheel_radius>
+          </wheel>
+        </xacro:macro>
+        <xacro:slip_wheel link="front_left_wheel_link"/>
+        <xacro:slip_wheel link="front_right_wheel_link"/>
+        <xacro:slip_wheel link="rear_left_wheel_link"/>
+        <xacro:slip_wheel link="rear_right_wheel_link"/>
+      </plugin>
+    </gazebo>
+  </xacro:if>
+  <!-- ==================================================================
        IMU
        Noise set for a consumer MEMS part (BNO055 / ICM-20948 class). Note the
