Commit message: The pod camera was imaging the world sideways; confirm now converges
THE POD CAMERA WAS MOUNTED ROLLED 90 DEGREES, at every arm pose, and had been
since the pod was added. arm_wrist_link's own frame is rolled about its forward
axis - its +Z points along the robot's +Y - so a camera mounted square to that
link produces an image whose RIGHT is the robot's FORWARD direction and whose
DOWN is the robot's LEFT. Nothing downstream can undo it: the pod sits before
wrist_roll deliberately, so the image never rolls.

That inverted the meaning of the one number three control loops are built on.
Every consumer - this repo's coordinator, and trash_vision, which we do not own
- reads `horizontal_error` as BEARING. Sideways it is RANGE, and bearing hides
in the vertical coordinate.

It failed in the worst available way: silently, and while looking healthy. The
detector reported plausible bounding boxes, the arm tracked its commanded pan to
1.3 mrad, the range sat squarely in the grasp window - and the loops simply
never converged. Measured off the URDF at confirm_pose before the fix: moving
the target 1 m sideways changed horizontal error by 0.000, and shoulder_pan, the
joint the aim loop uses to null that error, had first-order authority over it of
exactly zero. The response is quadratic with its peak at pan 0, so the previous
commit's "overshooting loop, suspect aim_gain" reading was wrong. There was
nothing to converge with. No gain would have worked.

Fixed by rolling the camera mount +90 deg. This is a rotation about the shared
view axis, so the ToF ray does not move and the two stay aimed together - the
pod_aim_rpy investigation in Task 5b is untouched. After: 1 m sideways moves
horizontal error by 3.124, and d(error)/d(pan) is -0.431 /rad at confirm_pose,
-0.636 at search_pose. Image up is now the robot's forward direction.

scripts/verify_pod_orientation.py pins all of it off the URDF, no simulator.

TWO CONSEQUENT FIXES:

- The aim loop integrates PLUS, not minus. With authority of -0.431 /rad a
  positive pan step reduces a positive error; subtracting walks the pan into a
  joint limit. The sign was genuinely unknowable before, the derivative being
  zero. aim_gain 1.0 closes 43% of the error per tick; 2.32 would be deadbeat.

- GRASP HEIGHT COMES FROM THE GROUND PLANE, NOT THE ToF. The ToF is a single ray
  and at confirm_pose it lands beside the litter, so the point it produces sits
  on the ground - measured, two of three targets came out 1.2 and 1.5 mm below
  it, which is the ground read to within its own noise. Litter rests on the
  ground, so the ray supplies bearing and radius and the ground supplies height.
  Mount height is read from tf, not written down.

  And the grasp height is 50 mm, NOT the arm's lowest reachable 35.4 mm. That
  figure sits on the singular edge of the workspace, where the radial window at
  a straight-down approach is 19 mm - tighter than the base can be placed. The
  window is a cliff: 40 mm gives 72 mm of it, 50 mm gives 123 mm. Relaxing the
  approach angle does not help; the whole -90..-87 deg range unions to 24 mm.
  This retires the "~50 mm band" figure in the progress notes.

RESULT, over two full runs. APPROACHING -> CONFIRMING -> PICKING now fires
repeatedly - seven times across the two runs, having never fired once before.
Confirmation settles in 0.5-1.2 s with bearing error driven to zero (-0.141 ->
-0.020, and 0.009 on another approach).

STILL FAILING: no grasp is solvable yet, but for a different and fully measured
reason. Nothing nulls RANGE. The gate into CONFIRMING tests apparent size and
horizontal centring, neither of which constrains radius, so the base stops where
it stops - the four grasp targets came out at r = 0.200, 0.039, 0.015 and 0.070
against a reachable band of 0.075-0.198. Two missed the edge by 2 and 5 mm.

The signal for that loop now exists, which it did not before this commit:
vertical image error IS the radial direction. At the grasp plane the band spans
vertical error +0.4655 (near edge) to -0.0828 (far edge), centred +0.1862 - a
wide, comfortable target. Creeping the base on it is the next step.

67 tests pass. Nothing in the pure modules changed.

Co-Authored-By: Claude Opus 5 <noreply@anthropic.com>

File: src/drivebase_description/urdf/drivebase.urdf.xacro (robot description, xacro)
@@ -301,4 +301,28 @@
          and the localisation maths assumes exactly that. -->
     <xacro:property name="pod_aim_rpy" value="0 0 0"/>
+    <!-- The camera is mounted rolled 90 degrees. The ToF is not, and does not
+         need to be: this is a rotation about the shared view axis, so the ray
+         does not move by even a rounding error and the two stay aimed together.
+         WHY. arm_wrist_link's own frame is rolled 90 degrees about its forward
+         axis - its +Z points along the robot's +Y, not up. Mounting the camera
+         square to that link therefore produces an image whose RIGHT is the
+         robot's FORWARD direction and whose DOWN is the robot's LEFT. The image
+         is sideways, at every arm pose, and constant, because the pod sits
+         before wrist_roll and nothing in the chain can roll it back.
+         That is not cosmetic. Every consumer - this repo's coordinator, and
+         trash_vision, which we do not own - reads `horizontal_error` as BEARING.
+         Sideways, it is RANGE instead, and bearing hides in the vertical
+         coordinate. Measured at confirm_pose before this roll: moving the target
+         1 m sideways changed horizontal error by 0.000, while shoulder_pan - the
+         joint the aim loop uses to null that error - had a first-order authority
+         over it of exactly zero (the response is quadratic, peaking at pan 0).
+         The confirm loop could not converge because there was nothing to
+         converge with.
+         With the roll: 1 m sideways moves horizontal error by 3.124, and
+         d(error)/d(pan) is -0.431 /rad at confirm_pose, -0.636 at search_pose.
+         Image up is the robot's forward direction, which is the conventional
+         orientation for a downward-looking camera and the one trash_vision
+         assumes. See scripts/verify_pod_orientation.py, which pins all of it. -->
+    <xacro:property name="pod_camera_roll" value="${pi/2}"/>
     <link name="pod_camera_link">
       <xacro:sensor_inertia/>
@@ -307,5 +331,5 @@
       <parent link="arm_wrist_link"/>
       <child  link="pod_camera_link"/>
-      <origin xyz="${pod_camera_xyz}" rpy="${pod_aim_rpy}"/>
+      <origin xyz="${pod_camera_xyz}" rpy="${pod_camera_roll} 0 0"/>
     </joint>
     <!-- ROS optical convention: z forward, x right, y down. Image pipelines and

Commit message: Measure the arm workspace at a 224 mm mount, without adopting it
THE DEFAULT IS UNCHANGED. arm_mount_height is a new xacro arg defaulting to
0.260, so the built configuration is exactly what it was and reverting is
deleting an override rather than editing geometry. Verified both ways:
arm_base_link lands at 260.0 mm with no argument and 224.0 mm with one.

WHY 224 mm IS INTERESTING. The reach floor is 224.4 mm below the mount wherever
the mount is, so at 260 mm the gripper bottoms out 35.6 mm above the ground and
cannot touch it. Flat litter is not hard to pick up, it is outside the
workspace - and litter_wrapper in the test field is 12 mm tall.

What governs tolerance is depth below the mount, not mount height, and radial
tolerance collapses as the target nears the reach floor:

  grasp height     band at 260 mm    band at 224 mm
     0 mm (ground)   out of reach       32 mm
    12 mm (wrapper)  OUT OF REACH      115 mm
    50 mm (a can)         123 mm       211 mm

shoulder_lift's margin to its +1.745 limit at band centre goes from +0.136 rad
to +0.448 - the arm stops working at the end of its travel everywhere it can
grasp, which is what section 5 of arm_workspace.md is really describing.

Raising grasp_height in software is geometrically identical to lowering the
mount, but it is capped by the litter and cannot help the wrapper at all. That
is the entire argument for the bracket.

Nothing blocks it. The ultrasonic band keeps 24.0 mm of clearance (the arm base
extends 2.4 mm below its mount point and 69.6 mm above); the coordinator parks
at search_pose, whose tip is 651 mm up; ground clearance and wheels are
unaffected. Below ~215 mm the sensor band does start to bind.

THESE ARE IDEAL COMMANDED KINEMATICS AND MUST NOT BE PASTED INTO
coordinator.yaml. They exclude the droop of section 5, and at both calibrated
poses the recorded sim figures differ in exactly the direction droop predicts -
search_pose reads 1.08-1.14 m against an FK 1.021, confirm_pose 0.2716 against
an FK 0.284. That agreement is the cross-check, not a licence to substitute.

Section 7 of arm_workspace.md lists every figure that moves, and the three
steps to put it back. Sections 1-6 remain the record of the 260 mm build and
are not superseded.

Also adds the capture rig behind the pose photographs, and the photographs. Two
notes worth not rediscovering, both in the script's docstring: Gazebo's
/gui/screenshot replies `data: true` and writes no file, and `import` fails on
this Wayland session where `grim` works.

67 tests pass; the pod-orientation guard passes. Neither depends on mount
height, so both passing after a revert confirms nothing drifted.

Co-Authored-By: Claude Opus 5 <noreply@anthropic.com>

File: src/drivebase_description/urdf/drivebase.urdf.xacro (robot description, xacro)
@@ -213,5 +213,11 @@
        link's own 87 mm height is accounted for.
        On the top plane (460 mm) the arm could not reach the ground at all. -->
-  <xacro:property name="arm_mount_z" value="0.200"/>  <!-- 260 mm above ground -->
+  <!-- Height above GROUND, so the trade study reads in the units it is argued
+       in. Everything the coordinator is calibrated on was measured at 0.260 -
+       see docs/arm_workspace.md section 7 before changing it, which lists every
+       figure that moves and how to put them back. -->
+  <xacro:arg name="arm_mount_height" default="0.260"/>
+  <xacro:property name="arm_mount_z"
+                  value="${$(arg arm_mount_height) - wheel_radius}"/>
   <link name="arm_mount_link">
     <xacro:sensor_inertia/>
